File: kicad/solarwetterstation/solarwetterstation.sch (KiCad schematic (older format))
At the start: 20 parts, among them J1 Conn_01x02_Male, J2 Conn_01x02_Male, J3 Conn_01x08_Male, J4 Conn_01x08_Male, J5 Conn_01x08_Male, J6 Conn_01x08_Male, U1 LM317_TO-220, U2 my_BME280, U3 ESP-12F, U4 1085

Commit message: änderungen vor rechner reinstall
Parts:
- J1, J2: footprint (none) -> TerminalBlock:TerminalBlock_Altech_AK300-2_P5.00mm
- J3, J4, J5, J6: footprint (none) -> Connector_PinHeader_2.54mm:PinHeader_1x08_P2.54mm_Vertical
- R1, R2, R3, R4, R5, R6, R7, R8, R9: footprint (none) -> Resistor_THT:R_Axial_DIN0207_L6.3mm_D2.5mm_P10.16mm_Horizontal
- U2: footprint Package_LGA:Bosch_LGA-8_2.5x2.5mm_P0.65mm_ClockwisePinNumbering -> (none)
- U3: footprint (none) -> ESP8266:ESP-12E
- U4: footprint MODULE_1085 -> (none)
Changed lines of the file:
@@
 F 0 "R9" H 9420 5546 50  0000 L CNN
 F 1 "100K" H 9420 5455 50  0000 L CNN
-F 2 "" V 9280 5500 50  0001 C CNN
+F 2 "Resistor_THT:R_Axial_DIN0207_L6.3mm_D2.5mm_P10.16mm_Horizontal" V 9280 5500 50  0001 C CNN
 F 3 "~" H 9350 5500 50  0001 C CNN
 	1    9350 5500
@@
 F 0 "R8" H 9420 5046 50  0000 L CNN
 F 1 "220K" H 9420 4955 50  0000 L CNN
-F 2 "" V 9280 5000 50  0001 C CNN
+F 2 "Resistor_THT:R_Axial_DIN0207_L6.3mm_D2.5mm_P10.16mm_Horizontal" V 9280 5000 50  0001 C CNN
 F 3 "~" H 9350 5000 50  0001 C CNN
 	1    9350 5000
@@
 F 0 "R1" V 3293 2800 50  0000 C CNN
 F 1 "470" V 3384 2800 50  0000 C CNN
-F 2 "" V 3430 2800 50  0001 C CNN
+F 2 "Resistor_THT:R_Axial_DIN0207_L6.3mm_D2.5mm_P10.16mm_Horizontal" V 3430 2800 50  0001 C CNN
 F 3 "~" H 3500 2800 50  0001 C CNN
 	1    3500 2800
@@
 F 0 "R2" V 3593 2800 50  0000 C CNN
 F 1 "47" V 3684 2800 50  0000 C CNN
-F 2 "" V 3730 2800 50  0001 C CNN
+F 2 "Resistor_THT:R_Axial_DIN0207_L6.3mm_D2.5mm_P10.16mm_Horizontal" V 3730 2800 50  0001 C CNN
 F 3 "~" H 3800 2800 50  0001 C CNN
 	1    3800 2800
@@
 F 0 "R3" V 3893 2800 50  0000 C CNN
 F 1 "10" V 3984 2800 50  0000 C CNN
-F 2 "" V 4030 2800 50  0001 C CNN
+F 2 "Resistor_THT:R_Axial_DIN0207_L6.3mm_D2.5mm_P10.16mm_Horizontal" V 4030 2800 50  0001 C CNN
 F 3 "~" H 4100 2800 50  0001 C CNN
 	1    4100 2800
@@
 F 0 "R5" V 5007 3200 50  0000 C CNN
 F 1 "220" V 4916 3200 50  0000 C CNN
-F 2 "" V 4730 3200 50  0001 C CNN
+F 2 "Resistor_THT:R_Axial_DIN0207_L6.3mm_D2.5mm_P10.16mm_Horizontal" V 4730 3200 50  0001 C CNN
 F 3 "~" H 4800 3200 50  0001 C CNN
 	1    4800 3200
@@
 F 0 "R4" V 4293 3200 50  0000 C CNN
 F 1 "20" V 4384 3200 50  0000 C CNN
-F 2 "" V 4430 3200 50  0001 C CNN
+F 2 "Resistor_THT:R_Axial_DIN0207_L6.3mm_D2.5mm_P10.16mm_Horizontal" V 4430 3200 50  0001 C CNN
 F 3 "~" H 4500 3200 50  0001 C CNN
 	1    4500 3200
@@
 F 0 "J1" H 2758 2281 50  0000 C CNN
 F 1 "Conn_01x02_Male" H 2758 2190 50  0000 C CNN
-F 2 "" H 2650 2100 50  0001 C CNN
+F 2 "TerminalBlock:TerminalBlock_Altech_AK300-2_P5.00mm" H 2650 2100 50  0001 C CNN
 F 3 "~" H 2650 2100 50  0001 C CNN
 	1    2650 2100
@@
 F 0 "J2" H 2858 5581 50  0000 C CNN
 F 1 "Conn_01x02_Male" H 2858 5490 50  0000 C CNN
-F 2 "" H 2750 5400 50  0001 C CNN
+F 2 "TerminalBlock:TerminalBlock_Altech_AK300-2_P5.00mm" H 2750 5400 50  0001 C CNN
 F 3 "~" H 2750 5400 50  0001 C CNN
 	1    2750 5400
@@
 F 0 "U3" H 8000 2265 50  0000 C CNN
 F 1 "ESP-12F" H 8000 2174 50  0000 C CNN
-F 2 "" H 8000 1500 50  0001 C CNN
+F 2 "ESP8266:ESP-12E" H 8000 1500 50  0001 C CNN
 F 3 "" H 8000 1500 50  0001 C CNN
 	1    8000 1500
@@
 F 0 "R6" H 6680 3254 50  0000 R CNN
 F 1 "10K" H 6680 3345 50  0000 R CNN
-F 2 "" V 6680 3300 50  0001 C CNN
+F 2 "Resistor_THT:R_Axial_DIN0207_L6.3mm_D2.5mm_P10.16mm_Horizontal" V 6680 3300 50  0001 C CNN
 F 3 "~" H 6750 3300 50  0001 C CNN
 	1    6750 3300
@@
 F 0 "R7" V 8993 3550 50  0000 C CNN
 F 1 "10K" V 9084 3550 50  0000 C CNN
-F 2 "" V 9130 3550 50  0001 C CNN
+F 2 "Resistor_THT:R_Axial_DIN0207_L6.3mm_D2.5mm_P10.16mm_Horizontal" V 9130 3550 50  0001 C CNN
 F 3 "~" H 9200 3550 50  0001 C CNN
 	1    9200 3550
@@
 F 0 "U4" V 8004 5630 50  0000 L CNN
 F 1 "1085" V 8095 5630 50  0000 L CNN
-F 2 "MODULE_1085" H 8050 5200 50  0001 L BNN
+F 2 "" H 8050 5200 50  0001 L BNN
 F 3 "" H 8050 5200 50  0001 L BNN
 F 4 "N/A" H 8050 5200 50  0001 L BNN "MAXIMUM_PACKAGE_HEIGHT"
@@
 F 0 "U2" H 4770 5146 50  0000 R CNN
 F 1 "my_BME280" H 4770 5055 50  0000 R CNN
-F 2 "Package_LGA:Bosch_LGA-8_2.5x2.5mm_P0.65mm_ClockwisePinNumbering" H 6700 4650 50  0001 C CNN
+F 2 "" H 6700 4650 50  0001 C CNN
 F 3 "https://ae-bst.resource.bosch.com/media/_tech/media/datasheets/BST-BME280-DS002.pdf" H 5200 4900 50  0001 C CNN
 	1    5200 5100
@@
 F 0 "J4" H 7622 3224 50  0000 R CNN
 F 1 "Conn_01x08_Male" H 7622 3133 50  0000 R CNN
-F 2 "" H 7650 3250 50  0001 C CNN
+F 2 "Connector_PinHeader_2.54mm:PinHeader_1x08_P2.54mm_Vertical" H 7650 3250 50  0001 C CNN
 F 3 "~" H 7650 3250 50  0001 C CNN
 	1    7650 3250
@@
 F 0 "J5" H 8658 3731 50  0000 C CNN
 F 1 "Conn_01x08_Male" H 8658 3640 50  0000 C CNN
-F 2 "" H 8550 3250 50  0001 C CNN
+F 2 "Connector_PinHeader_2.54mm:PinHeader_1x08_P2.54mm_Vertical" H 8550 3250 50  0001 C CNN
 F 3 "~" H 8550 3250 50  0001 C CNN
 	1    8550 3250
@@
 F 0 "J3" H 7008 1981 50  0000 C CNN
 F 1 "Conn_01x08_Male" H 7008 1890 50  0000 C CNN
-F 2 "" H 6900 1500 50  0001 C CNN
+F 2 "Connector_PinHeader_2.54mm:PinHeader_1x08_P2.54mm_Vertical" H 6900 1500 50  0001 C CNN
 F 3 "~" H 6900 1500 50  0001 C CNN
 	1    6900 1500
@@
 F 0 "J6" H 9072 1474 50  0000 R CNN
 F 1 "Conn_01x08_Male" H 9072 1383 50  0000 R CNN
-F 2 "" H 9100 1500 50  0001 C CNN
+F 2 "Connector_PinHeader_2.54mm:PinHeader_1x08_P2.54mm_Vertical" H 9100 1500 50  0001 C CNN
 F 3 "~" H 9100 1500 50  0001 C CNN
 	1    9100 1500
