File: kicad/solarwetterstation/solarwetterstationV2.sch (KiCad schematic (older format))
At the start: 20 parts, among them J1 Conn_01x02_Male, J2 Conn_01x02_Male, J3 Conn_01x08_Male, J4 Conn_01x08_Male, J5 Conn_01x08_Male, J6 Conn_01x08_Male, U1 LM317_TO-220, U2 my_BME280, U3 ESP-12F, U4 1085

Commit message: änderungen vor rechner reinstall
Parts:
- removed J3, J6: Conn_01x08_Male, symbol Connector:Conn_01x08_Male
- removed U2: my_BME280, Package_LGA:Bosch_LGA-8_2.5x2.5mm_P0.65mm_ClockwisePinNumbering, symbol MySensor:my_BME280
- removed U3: ESP-12F, symbol ESP8266:ESP-12F
- removed U4: 1085, MODULE_1085, symbol 1085:1085
- added U2: BME280, dele72:myBME280, symbol deleSymbols:BME280
- added U4: ADS1115, dele72:myADS1115, symbol deleSymbols:ADS1115
- J1, J2: footprint (none) -> TerminalBlock:TerminalBlock_Altech_AK300-2_P5.00mm
- J4, J5: footprint (none) -> Connector_PinHeader_2.54mm:PinHeader_1x08_P2.54mm_Vertical
- R1, R2, R3, R4, R5, R6, R7, R8, R9: footprint (none) -> Resistor_THT:R_Axial_DIN0207_L6.3mm_D2.5mm_P10.16mm_Horizontal
Connections:
- net +3.3VADC: now also U2.6 (VCC), U4.10 (VDD), U4.3 (AIN1)
- net GND: now also U2.5 (GND), U4.9 (GND)
- net at R8.2, R9.1: now also U4.4 (AIN0)
- net at J5.4 (Pin_4): now also U2.3 (SDA), U4.7 (SDA)
- net at J5.3 (Pin_3): now also U2.4 (SCL), U4.8 (SCL)
- no-connect marks 22 -> 16
Other:
- note added: "(1) REST"
- note added: "(10) GPIO15"
- note added: "(11) GPIO02"
- note added: "(12) GPIO0"
- note added: "(13) GPIO4"
- note added: "(14) GPIO5"
- note added: "(15) RXD"
- note added: "(16) TXD"
- note added: "(17) CS0"
- note added: "(18) MISO"
- note added: "(19) GPIO9"
- note added: "(2) ADC"
- note added: "(20) GPIO10"
- note added: "(21) MOSI"
- note added: "(22) SCLK"
- note added: "(3) CH_PD"
- note added: "(4) GPIO16"
- note added: "(5) GPIO14"
- note added: "(6) GPIO12"
- note added: "(7) GPIO13"
- note added: "(8) VCC"
- note added: "(9) GND"
- note added: "ESP-12F"
- note added: "ESP-12F Conn."
